File: eclipse-lamp/electronics/core/eclipse-core.kicad_sch (KiCad schematic)
At the start: 66 parts, among them J1 USB-C 16P, J2 TO HALO, J3 UPDI, U1 CH224K, U2 AMS1117-3.3, U3 ATtiny1616-S, U4 TPS61165, U5 TPS61165, U6 TPS61165, U7 TPS61165

Commit message: ECLIPSE: light emanates through the body (diffusion redesign)
- Halo is now a hollow light-diffusing PMMA body under a thin graphite cap;
  the LED board fires down into it, so the underside gives task light and
  the walls glow with a soft falloff toward the cap
- Base gains a glowing opal band lit by an internal light chamber (white
  steel reflector/weight); steel plinth keeps the CoG 40 mm inside the edge
- Core board: 8 rim 2835 LEDs + AO3400A on PC0 (TCD0 PWM) for the base glow;
  schematic fully wired (no labels), ERC/DRC clean, re-routed, fab re-exported
- Renders: glow-material shader, new close-up and night-glow shots
- BOM, README and design notes updated (thermal/PMMA margin, stability)

Co-Authored-By: Claude Opus 5.5 <noreply@anthropic.com>
Claude-Session: https://claude.ai/code/session_01UC4Dpjx8nsVkJqTcucsgsg
Parts:
- added D10, D11, D12, D13, D14, D7, D8, D9: 2700K, LED_SMD:LED_PLCC_2835, symbol Device:LED
- added Q1: AO3400A, Package_TO_SOT_SMD:SOT-23, symbol Transistor_FET:AO3400A
- added R18, R19, R20, R21, R22, R23, R24, R25, R26: 100, Resistor_SMD:R_0603_1608Metric, symbol Device:R
- added R27: 100k, Resistor_SMD:R_0603_1608Metric, symbol Device:R
Connections:
- net +3V3: now also R18.1, R19.1, R20.1, R21.1, R22.1, R23.1, R24.1, R25.1
- net GND: now also Q1.2 (S), R27.2
- net at U3.12 (PC0): now also R26.1
- new net: D10.1 (K), D11.1 (K), D12.1 (K), D13.1 (K), D14.1 (K), D7.1 (K), D8.1 (K), D9.1 (K), Q1.3 (D)
- new net: D7.2 (A), R18.2
- new net: D10.2 (A), R21.2
- new net: D12.2 (A), R23.2
- new net: Q1.1 (G), R26.2, R27.1
- new net: D11.2 (A), R22.2
- new net: D14.2 (A), R25.2
- new net: D9.2 (A), R20.2
- new net: D13.2 (A), R24.2
- new net: D8.2 (A), R19.2
- no-connect marks 11 -> 10
Other:
- note added: "11 BODY GLOW (lights the opal base band) + MECHANICAL"
- note added: "PC0 = TCD0 WOC PWM: breathing night-glow through the base"
- note removed: "11 MECHANICAL"
- moved on the sheet: H1, H2, H3

Commit message: ECLIPSE Tree: an intricately branched cedar elm whose 800 leaves are 0402 LEDs
- Procedural cedar-elm generator (seeded): S-curved trunk, burl fork, 4 limbs,
  75 branches + 189 spur twigs, pipe-model diameters, drooping branchlets
- New sprig flex PCB: 2-layer polyimide cedar-elm spray, 20 x 0402 LED leaves
  in parallel, outline grown around the copper; shared layout with the 3D model
- New hub PCB (in the burl): 40 sprig lands, four 10-sprig series chains, NTC;
  same 10-wire harness pinout so the core board circuit is unchanged
- Halo ring board retired; all schematics fully wired, ERC/DRC/parity clean
- CAD, BOM (~$72), wiring map, README/design notes and Cycles renders updated

Co-Authored-By: Claude Opus 5.5 <noreply@anthropic.com>
Claude-Session: https://claude.ai/code/session_01UC4Dpjx8nsVkJqTcucsgsg
Parts:
- J2: value TO HALO -> TO HUB
Other:
- note added: "10 TRUNK HARNESS (to the tree hub)"
- note added: "1:1 harness to hub J1 (up the trunk)"
- note removed: "10 HALO HARNESS"
- note removed: "1:1 harness to halo J1 (through the stem)"
- title: ECLIPSE - Core board (base): power, drivers, touch MCU -> ECLIPSE Tree - Core board (base): power, drivers, touch MCU
Changed lines of the file:
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@@
 	(paper "A2")
 	(title_block
-		(title "ECLIPSE - Core board (base): power, drivers, touch MCU")
+		(title "ECLIPSE Tree - Core board (base): power, drivers, touch MCU")
 		(date "2026-10-07")
 		(rev "A")
@@
 		(comment 1 "USB-C PD 9 V sink, 4ch boost CC LED drivers, ATtiny1616 capacitive touch")
 		(comment 2 "Board: 2 layers, 1.6 mm FR4, 1 oz, matte black mask, ENIG")
-		(comment 3 "Mates with eclipse-halo ring board through J2 / 10-wire JST-PH harness (1:1)")
+		(comment 3 "J2: 10-wire harness up the trunk to the eclipse-hub board (1:1)")
 	)
 	(text "1  USB-C POWER DELIVERY SINK (requests 9 V)"
@@
 		)
 	)
-	(text "10  HALO HARNESS"
+	(text "10  TRUNK HARNESS (to the tree hub)"
 		(exclude_from_sim no)
 		(at 384.27 298.64 0)
@@
 		)
 	)
-	(text "1:1 harness to halo J1 (through the stem)"
+	(text "1:1 harness to hub J1 (up the trunk)"
 		(exclude_from_sim no)
 		(at 386.08 391.16 0)
@@
 			)
 		)
-		(property "Value" "TO HALO"
+		(property "Value" "TO HUB"
 			(at 429.26 355.6 0)
 			(effects
