File: eclipse-lamp/electronics/core/eclipse-core.kicad_pcb (KiCad board)
At the start: 2 copper layers, 135.2 x 123.1 mm, 66 parts, among them J1 USB-C 16P, J2 TO HALO, J3 UPDI, U1 CH224K, U2 AMS1117-3.3, U3 ATtiny1616-S, U4 TPS61165, U5 TPS61165, U6 TPS61165, U7 TPS61165

Commit message: ECLIPSE: light emanates through the body (diffusion redesign)
- Halo is now a hollow light-diffusing PMMA body under a thin graphite cap;
  the LED board fires down into it, so the underside gives task light and
  the walls glow with a soft falloff toward the cap
- Base gains a glowing opal band lit by an internal light chamber (white
  steel reflector/weight); steel plinth keeps the CoG 40 mm inside the edge
- Core board: 8 rim 2835 LEDs + AO3400A on PC0 (TCD0 PWM) for the base glow;
  schematic fully wired (no labels), ERC/DRC clean, re-routed, fab re-exported
- Renders: glow-material shader, new close-up and night-glow shots
- BOM, README and design notes updated (thermal/PMMA margin, stability)

Co-Authored-By: Claude Opus 5.5 <noreply@anthropic.com>
Claude-Session: https://claude.ai/code/session_01UC4Dpjx8nsVkJqTcucsgsg
Parts:
- added D10: 2700K, LED_SMD:LED_PLCC_2835, B.Cu at (167.0, 205.5)
- added D11: 2700K, LED_SMD:LED_PLCC_2835, B.Cu at (130.2, 204.5)
- added D12: 2700K, LED_SMD:LED_PLCC_2835, B.Cu at (99.8, 179.0)
- added D13: 2700K, LED_SMD:LED_PLCC_2835, B.Cu at (94.0, 135.0)
- added D14: 2700K, LED_SMD:LED_PLCC_2835, B.Cu at (102.5, 116.7)
- added D7: 2700K, LED_SMD:LED_PLCC_2835, B.Cu at (169.8, 95.5)
- added D8: 2700K, LED_SMD:LED_PLCC_2835, B.Cu at (201.2, 122.8)
- added D9: 2700K, LED_SMD:LED_PLCC_2835, B.Cu at (201.2, 177.2)
- added Q1: AO3400A, Package_TO_SOT_SMD:SOT-23, B.Cu at (134.0, 138.0)
- added R18: 100, Resistor_SMD:R_0603_1608Metric, B.Cu at (168.3, 99.7)
- added R19: 100, Resistor_SMD:R_0603_1608Metric, B.Cu at (197.2, 124.9)
- added R20: 100, Resistor_SMD:R_0603_1608Metric, B.Cu at (197.2, 175.1)
- added R21: 100, Resistor_SMD:R_0603_1608Metric, B.Cu at (165.6, 201.2)
- added R22: 100, Resistor_SMD:R_0603_1608Metric, B.Cu at (131.7, 200.3)
- added R23: 100, Resistor_SMD:R_0603_1608Metric, B.Cu at (103.7, 176.8)
- added R24: 100, Resistor_SMD:R_0603_1608Metric, B.Cu at (98.3, 136.2)
- added R25: 100, Resistor_SMD:R_0603_1608Metric, B.Cu at (106.2, 119.3)
- added R26: 100, Resistor_SMD:R_0603_1608Metric, B.Cu at (134.0, 142.0)
- added R27: 100k, Resistor_SMD:R_0603_1608Metric, B.Cu at (130.5, 142.0)
Connections:
- U3 pad 12: unconnected-(U3-PC0-Pad12) -> Net-(U3-PC0)
Routing:
- net Net-(D10-K): track 0.00 -> 349.7 mm, vias 0 -> 2
- net +3V3: track 136.5 -> 374.1 mm
- net GND: track 476.6 -> 596.7 mm, vias 1 -> 2
- net Net-(U3-PA7): track 37.2 -> 67.1 mm, vias 2 -> 0
- net Net-(U3-PC0): track 0.00 -> 26.4 mm, vias 0 -> 2
- net Net-(J2-Pin_7): track 129.4 -> 150.9 mm
- net Net-(J1-CC1): track 16.9 -> 36.8 mm, vias 2 -> 0
- net Net-(J1-CC2): track 16.6 -> 32.7 mm, vias 2 -> 0
- net Net-(U3-PB1): track 94.7 -> 110.2 mm, vias 4 -> 3
- net Net-(J2-Pin_4): track 75.2 -> 87.9 mm
- net Net-(U3-PA1): track 21.0 -> 11.2 mm
- net Net-(Q1-G): track 0.00 -> 7.42 mm
- net Net-(U1-VDD): track 13.9 -> 21.1 mm
- net Net-(U4-COMP): track 5.69 -> 12.2 mm
- net Net-(U5-COMP): track 12.2 -> 5.75 mm
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
Commit message: ECLIPSE Tree: an intricately branched cedar elm whose 800 leaves are 0402 LEDs
- Procedural cedar-elm generator (seeded): S-curved trunk, burl fork, 4 limbs,
  75 branches + 189 spur twigs, pipe-model diameters, drooping branchlets
- New sprig flex PCB: 2-layer polyimide cedar-elm spray, 20 x 0402 LED leaves
  in parallel, outline grown around the copper; shared layout with the 3D model
- New hub PCB (in the burl): 40 sprig lands, four 10-sprig series chains, NTC;
  same 10-wire harness pinout so the core board circuit is unchanged
- Halo ring board retired; all schematics fully wired, ERC/DRC/parity clean
- CAD, BOM (~$72), wiring map, README/design notes and Cycles renders updated

Co-Authored-By: Claude Opus 5.5 <noreply@anthropic.com>
Claude-Session: https://claude.ai/code/session_01UC4Dpjx8nsVkJqTcucsgsg
Parts:
- J2: value TO HALO -> TO HUB
Other:
- board text added: "TO TREE HUB"
- board text removed: "TO HALO"
Changed lines of the file:
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@@
 			)
 		)
-		(property "Value" "TO HALO"
+		(property "Value" "TO HUB"
 			(at 0 -5.8 0)
 			(layer "B.Fab")
@@
 		)
 	)
-	(gr_text "TO HALO"
+	(gr_text "TO TREE HUB"
 		(at 125 109.5 0)
 		(layer "B.SilkS")
