File: eclipse-lamp/electronics/hub/eclipse-hub.kicad_sch (KiCad schematic)
At the start: 42 parts, among them J1 TO CORE J2

Commit message: ECLIPSE Tree: thick glowing trunk, 5x crown, fibre-lit samaras, hub light engine
- Tree: 44 mm cast-bronze trunk shell around a PMMA light-guide core with
  glowing bark fissures, 6 buttress roots, D68 burl, 73 branches + 1222 spur
  twigs, 657 end-glow fibre tips with diffusing samaras
- Hub: D56 two-sided light engine (8 LEDs into the trunk core, 8 into the
  fibre bundles) as the first series element of each 100 mA chain; core
  board circuit unchanged; ERC/DRC/parity clean, all schematics wired
- Renders: fissure-glow bark shader, samaras, trunk close-up; BOM, docs

Co-Authored-By: Claude Opus 5.5 <noreply@anthropic.com>
Claude-Session: https://claude.ai/code/session_01UC4Dpjx8nsVkJqTcucsgsg
Parts:
- added D1, D10, D11, D12, D2, D3, D4, D9: 2700K, LED_SMD:LED_PLCC_2835, symbol Device:LED
- added D13, D14, D15, D16, D5, D6, D7, D8: 6500K, LED_SMD:LED_PLCC_2835, symbol Device:LED
Connections:
- net at S1.1 (Pin_1): now also D1.1 (K), D2.1 (K), D3.1 (K), D4.1 (K); no longer J1.3 (Pin_3)
- net at S11.1 (Pin_1): now also D5.1 (K), D6.1 (K), D7.1 (K), D8.1 (K); no longer J1.2 (Pin_2)
- net at S21.1 (Pin_1): now also D10.1 (K), D11.1 (K), D12.1 (K), D9.1 (K); no longer J1.8 (Pin_8)
- net at S31.1 (Pin_1): now also D13.1 (K), D14.1 (K), D15.1 (K), D16.1 (K); no longer J1.9 (Pin_9)
- new net: D10.2 (A), D11.2 (A), D12.2 (A), D9.2 (A), J1.8 (Pin_8)
- new net: D1.2 (A), D2.2 (A), D3.2 (A), D4.2 (A), J1.3 (Pin_3)
- new net: D5.2 (A), D6.2 (A), D7.2 (A), D8.2 (A), J1.2 (Pin_2)
- new net: D13.2 (A), D14.2 (A), D15.2 (A), D16.2 (A), J1.9 (Pin_9)
Other:
- note added: "CHAIN C1 (6500 K: light engine + 10 sprigs in series, 100 mA)"
- note added: "CHAIN C2 (6500 K: light engine + 10 sprigs in series, 100 mA)"
- note added: "CHAIN W1 (2700 K: light engine + 10 sprigs in series, 100 mA)"
- note added: "CHAIN W2 (2700 K: light engine + 10 sprigs in series, 100 mA)"
- note removed: "CHAIN C1 (6500 K, 10 sprigs in series, 100 mA)"
- note removed: "CHAIN C2 (6500 K, 10 sprigs in series, 100 mA)"
- note removed: "CHAIN W1 (2700 K, 10 sprigs in series, 100 mA)"
- note removed: "CHAIN W2 (2700 K, 10 sprigs in series, 100 mA)"
- title: ECLIPSE Tree - Hub board (sprig chaining, in the burl) -> ECLIPSE Tree - Hub light engine (in the burl)
- moved on the sheet: S1, S10, S11, S12, S13, S14, S15, S16, S17, S18, S19, S2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

Commit message: ECLIPSE Tree: regrow the tree so it reads as a real cedar elm
Space-colonisation crown in a lobed rounded envelope, pipe-model taper
from a 77 mm trunk through three leaders to 1,174 twigs, a smooth
tangent-lobed fork (the ball burl is gone; the hub sits in the fork
swelling), half-buried buttress roots, 21,770 light-diffusing film leaves,
smaller samaras, sprigs grafted inside the crown. Renderer blends the
wood into one remeshed body, adds translucent foliage and bark furrows.
Docs, BOM, wiring map and hub schematic title updated (ERC/DRC clean).

Co-Authored-By: Claude Opus 5.5 <noreply@anthropic.com>
Claude-Session: https://claude.ai/code/session_01UC4Dpjx8nsVkJqTcucsgsg
Other:
- title: ECLIPSE Tree - Hub light engine (in the burl) -> ECLIPSE Tree - Hub light engine (in the trunk fork)
Changed lines of the file:
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@@
 	(paper "A2")
 	(title_block
-		(title "ECLIPSE Tree - Hub light engine (in the burl)")
+		(title "ECLIPSE Tree - Hub light engine (in the trunk fork)")
 		(date "2026-10-07")
 		(rev "B")
 		(company "ECLIPSE desk lamp - open hardware")
 		(comment 1 "Per channel: 4 x 2835 (2 fibre / 2 trunk core) + 10 sprigs in series; crown NTC")
-		(comment 2 "Board: D56 mm, 2 layers 1.0 mm FR4, 1 oz, white mask (reflector), ENIG, in the burl")
+		(comment 2 "Board: D56 mm, 2 layers 1.0 mm FR4, 1 oz, white mask (reflector), ENIG, in the trunk fork")
 		(comment 3 "J1 = 10 trunk-wire lands, pinout identical to core J2")
 	)
